Commit message: modify xacro

File: tm_description/xacro/tm12_ecbpi.urdf.xacro (robot description, xacro)
@@ -1,8 +1,9 @@
 <?xml version="1.0"?>
-<robot xmlns:xacro="http://www.ros.org/wiki/xacro" name="tm12">
+<robot xmlns:xacro="http://www.ros.org/wiki/xacro" name="tm12_ecpbi">
   <xacro:arg name="ns" default="" />
   <xacro:arg name="prefix" default="" />
   <xacro:arg name="color" default="none" />
   <xacro:arg name="trans_hw_iface" default="hardware_interface/PositionJointInterface" />
+  <xacro:arg name="hand_link_name" default="ecpbi_base" />
   <xacro:include filename="$(find tm_description)/xacro/macro.gazebo.xacro" />
   <xacro:include filename="$(find tm_description)/xacro/macro.transmission.xacro" />
@@ -13,4 +14,9 @@
   <xacro:include filename="$(find tm_description)/xacro/macro.tm12-nominal.urdf.xacro" />
   <xacro:include filename="$(find tm_description)/xacro/schmalz_ecbpi_model_macro.xacro" />
+  <joint name="falange" type="fixed">
+    <parent link="flange" />
+    <child link="ecpbi_base" />
+    <origin xyz="0 0 0.1" rpy="0 0 0" />
+  </joint>
   <!--  -->
   <xacro:tmr_gazebo ns="$(arg ns)" prefix="$(arg prefix)" />
