Commit message: modify xacro

File: tm_description/xacro/schmalz_ecbpi_model_macro.xacro (robot description, xacro)
@@ -5,5 +5,5 @@
   <xacro:property name="joint_upper_limit" value="0.055" />
   <xacro:macro name="ecbpi_hand" params="hand_link_name robot_name">
-    <link name="${hand_link_name}">
+    <link name="ecpbi_base">
       <inertial>
         <mass value="0.745" />
@@ -47,5 +47,5 @@
     </link>
     <joint name="$hand__end_effector_joint" type="fixed">
-      <parent link="${hand_link_name}"/>
+      <parent link="ecpbi_base"/>
       <child link="ecbpi_end_effector"/>
       <origin xyz="0 0 ${0.13}" rpy="0 0 0"/>

File: tm_description/xacro/tm12_ecbpi.urdf.xacro (robot description, xacro)
@@ -14,9 +14,4 @@
   <xacro:include filename="$(find tm_description)/xacro/macro.tm12-nominal.urdf.xacro" />
   <xacro:include filename="$(find tm_description)/xacro/schmalz_ecbpi_model_macro.xacro" />
-  <joint name="falange" type="fixed">
-    <parent link="flange" />
-    <child link="ecpbi_base" />
-    <origin xyz="0 0 0.1" rpy="0 0 0" />
-  </joint>
   <!--  -->
   <xacro:tmr_gazebo ns="$(arg ns)" prefix="$(arg prefix)" />

Commit message: modify ecbpi xacro

File: tm_description/xacro/schmalz_ecbpi_model_macro.xacro (robot description, xacro)
@@ -12,7 +12,7 @@
       </inertial>
       <visual>
-        <origin xyz="0 0 0.095" rpy="0 0 0"/>
+        <origin xyz="0 0 0.0" rpy="0 0 0"/>
         <geometry>
-          <mesh filename="$(find tm_description)/meshes/ecbpi/visual/ecbpi.stl" scale="1.0 1.0 1.0"/>
+          <mesh filename="$(find tm_description)/meshes/ecbpi/visual/ecbpi.stl" scale="1000 1000 1000"/>
         </geometry>
         <material name="">

File: tm_description/xacro/tm12_ecbpi.urdf.xacro (robot description, xacro)
@@ -12,5 +12,5 @@
   <!-- you must modify 'macro.tm12-nominal.urdf.xacro' to 'user_defined.urdf.xacro'  -->
   <xacro:include filename="$(find tm_description)/xacro/macro.tm12-nominal.urdf.xacro" />
-  <xacro:include filename="/home/tak-mahal/ws_moveit2/src/tmr_ros2/tm_description/xacro/schmalz_ecbpi_model_macro.xacro" />
+  <xacro:include filename="$(find tm_description)/xacro/schmalz_ecbpi_model_macro.xacro" />
   <xacro:ecbpi_hand parent_link="flange" robot_name="tm12_ecbpi"/>
   <!--  -->

Commit message: modify tm12 packages

File: tm_description/xacro/schmalz_ecbpi_model_macro.xacro (robot description, xacro)
@@ -6,13 +6,13 @@
   <xacro:macro name="ecbpi_hand" params="parent_link robot_name">
     <link name="ecbpi_base">
-      <inertial>
+      <!--<inertial>
         <mass value="0.745" />
         <origin xyz="0 0.0 0.055" rpy="0 0 0" />
         <inertia ixx="0.003084" ixy="0.0" ixz="0.0" iyy="0.002999" iyz="0.0" izz="0.000546" />
-      </inertial>
+      </inertial>-->
       <visual>
-        <origin xyz="0 0 0.0" rpy="0 0 0"/>
+        <!--origin xyz="0 0 0.0" rpy="0 0 0"/-->
         <geometry>
-          <mesh filename="$(find tm_description)/meshes/ecbpi/visual/ecbpi.stl" scale="1000 1000 1000"/>
+          <mesh filename="file://$(find tm_description)/meshes/ecbpi/visual/ecbpi.dae" scale="1000 1000 1000"/>
         </geometry>
         <material name="">
@@ -20,5 +20,5 @@
         </material>
       </visual>
-      <visual>
+      <!--<visual>
         <origin xyz="0 0 ${0.015+0.095}" rpy="0 0 0"/>
         <geometry>
@@ -28,10 +28,10 @@
           <color rgba="1 1 1 1"/>
         </material>
-      </visual>
+      </visual>-->
       <collision>
         <!-- -0.095 + 0.102/2 = -0.044-->
-        <origin xyz="0 0 ${-0.044+0.095+0.014}" rpy="0 0 0"/>
+        <origin xyz="0 0 0" rpy="0 0 0"/>
         <geometry>
-          <cylinder radius="0.044" length="0.13"/>
+          <mesh filename="file://$(find tm_description)/meshes/ecbpi/collision/ecbpi_c.dae" scale="1000 1000 1000"/>
         </geometry>
       </collision>
@@ -40,5 +40,5 @@
       <parent link="${parent_link}"/>
       <child link="ecbpi_base"/>
-      <origin xyz="0 0 ${0.13}" rpy="0 0 0"/>
+      <origin xyz="0 0 0" rpy="0 0 ${0.5*pi}"/>
     </joint>
     <xacro:ecbpi_hand_gazebo robot_name="${robot_name}" />

Commit message: modify xacro

File: tm_description/xacro/schmalz_ecbpi_model_macro.xacro (robot description, xacro)
@@ -14,5 +14,5 @@
         <!--origin xyz="0 0 0.0" rpy="0 0 0"/-->
         <geometry>
-          <mesh filename="file://$(find tm_description)/meshes/ecbpi/visual/ecbpi.dae" scale="1000 1000 1000"/>
+          <mesh filename="file://$(find tm_description)/meshes/ecbpi/visual/ecbpi.dae" scale="1 1 1"/>
         </geometry>
         <material name="">
@@ -33,5 +33,5 @@
         <origin xyz="0 0 0" rpy="0 0 0"/>
         <geometry>
-          <mesh filename="file://$(find tm_description)/meshes/ecbpi/collision/ecbpi_c.dae" scale="1000 1000 1000"/>
+          <mesh filename="file://$(find tm_description)/meshes/ecbpi/collision/ecbpi_c.dae" scale="1 1 1"/>
         </geometry>
       </collision>

Commit message: update package

File: tm_description/xacro/schmalz_ecbpi_model_macro.xacro (robot description, xacro)
@@ -14,5 +14,5 @@
         <!--origin xyz="0 0 0.0" rpy="0 0 0"/-->
         <geometry>
-          <mesh filename="file://$(find tm_description)/meshes/ecbpi/visual/ecbpi.dae" scale="1 1 1"/>
+          <mesh filename="file://$(find tm_description)/meshes/ecbpi/visual/ecbpi.dae"/>
         </geometry>
         <material name="">
@@ -33,5 +33,5 @@
         <origin xyz="0 0 0" rpy="0 0 0"/>
         <geometry>
-          <mesh filename="file://$(find tm_description)/meshes/ecbpi/collision/ecbpi_c.dae" scale="1 1 1"/>
+          <mesh filename="file://$(find tm_description)/meshes/ecbpi/collision/ecbpi_c.dae"/>
         </geometry>
       </collision>
