Commit message: moidfy

File: tm_description/xacro/schmalz_ecbpi2_model_macro.xacro (robot description, xacro)
@@ -47,4 +47,12 @@
       <origin xyz="0 0 0" rpy="0 0 ${0.5*pi}"/>
     </joint>
+    <!--link name="ecbpi_tcp">
+      <origin xyz="0 -0.044 0.18" rpy="0 0 0"/>
+    </link>
+    <joint name="ecbpi_bast_to_tcp" type="fixed">
+      <parent link="ecbpi_base"/>
+      <child link="ecbpi_tcp"/>
+      <origin xyz = "0 0 0" rpy="0 0 0"/>
+    </joint-->
     <xacro:ecbpi_hand_gazebo robot_name="${robot_name}" />
   </xacro:macro>
