Commit message: 01211817_kyouyou

File: tm_description/xacro/schmalz_ecbpi3_model_macro.xacro (robot description, xacro)
@@ -41,4 +41,10 @@
         </geometry>
       </collision>
+      <collision>
+        <origin xyz="0.07 0 0.01" rpy="0 0 0"/>
+        <geometry>
+          <cylinder radius="0.04" length="0.1"/>
+        </geometry>
+      </collision>
     </link>
     <joint name="${parent_link}_to_ecbpi_joint" type="fixed">

Commit message: 01221920_kyouyou

File: tm_description/xacro/schmalz_ecbpi3_model_macro.xacro (robot description, xacro)
@@ -32,5 +32,5 @@
         <origin xyz="-0.044 0 0.05" rpy="0 0 0"/>
         <geometry>
-          <cylinder radius="0.08" length="0.1"/>
+          <cylinder radius="0.09" length="0.1"/>
         </geometry>
       </collision>
@@ -38,5 +38,5 @@
         <origin xyz="-0.044 0 0.14" rpy="0 0 0"/>
         <geometry>
-          <cylinder radius="0.025" length="0.08"/>
+          <cylinder radius="0.030" length="0.08"/>
         </geometry>
       </collision>

Commit message: 0227_honban

File: tm_description/xacro/schmalz_ecbpi3_model_macro.xacro (robot description, xacro)
@@ -12,5 +12,5 @@
       </inertial>-->
       <visual>
-        <!--origin xyz="0 0 0.0" rpy="0 0 0"/-->
+        <origin xyz="0 0 0.0" rpy="0 0 ${0.5*pi}"/>
         <geometry>
           <mesh filename="file://$(find tm_description)/meshes/ecbpi/visual/ecbpi.dae"/>
@@ -30,5 +30,5 @@
       </visual>-->
       <collision>
-        <origin xyz="-0.044 0 0.05" rpy="0 0 0"/>
+        <origin xyz="0 -0.044 0.05" rpy="0 0 0"/>
         <geometry>
           <cylinder radius="0.09" length="0.1"/>
@@ -36,5 +36,5 @@
       </collision>
       <collision>
-        <origin xyz="-0.044 0 0.14" rpy="0 0 0"/>
+        <origin xyz="0 -0.044 0.14" rpy="0 0 0"/>
         <geometry>
           <cylinder radius="0.030" length="0.08"/>
@@ -42,5 +42,5 @@
       </collision>
       <collision>
-        <origin xyz="0.07 0 0.01" rpy="0 0 0"/>
+        <origin xyz="0 0.07 0.01" rpy="0 0 0"/>
         <geometry>
           <cylinder radius="0.04" length="0.1"/>
@@ -51,5 +51,6 @@
       <parent link="${parent_link}"/>
       <child link="ecbpi_base"/>
-      <origin xyz="0 0 0" rpy="0 0 ${0.5*pi}"/>
+      <origin xyz="0 0 0" rpy="0 0 0"/>
+      <!--origin xyz="0 0 0" rpy="0 0 ${0.5*pi}"/-->
     </joint>
     <link name="ecbpi_tcp">
@@ -59,5 +60,6 @@
       <parent link="ecbpi_base"/>
       <child link="ecbpi_tcp"/>
-      <origin xyz = "-0.044 0 0.195" rpy="0 0 0"/>
+      <origin xyz = "0 -0.044 0.195" rpy="0 0 0"/>
+      <!--origin xyz = "-0.044 0 0.195" rpy="0 0 0"/-->
     </joint>
     <xacro:ecbpi_hand_gazebo robot_name="${robot_name}" />
