Commit message: add tm12_ecbpi_moveit_config

File: tm12_ecbpi_moveit_config/config/tm12_ecbpi.ros2_control.xacro (robot description, xacro)
@@ -1,5 +1,5 @@
 <?xml version="1.0"?>
 <robot xmlns:xacro="http://www.ros.org/wiki/xacro">
-    <xacro:macro name="tm12_ros2_control" params="name initial_positions_file">
+    <xacro:macro name="tm12_ecbpi_ros2_control" params="name initial_positions_file">
         <xacro:property name="initial_positions" value="${load_yaml(initial_positions_file)['initial_positions']}"/>
         <ros2_control name="${name}" type="system">

File: tm_description/xacro/schmalz_ecbpi_model_macro.xacro (robot description, xacro)
@@ -4,6 +4,6 @@
   <xacro:property name="joint_lower_limit" value="0.0" />
   <xacro:property name="joint_upper_limit" value="0.055" />
-  <xacro:macro name="ecbpi_hand" params="hand_link_name robot_name">
-    <link name="ecpbi_base">
+  <xacro:macro name="ecbpi_hand" params="parent_link robot_name">
+    <link name="ecbpi_base">
       <inertial>
         <mass value="0.745" />
@@ -36,37 +36,11 @@
         </geometry>
       </collision>
-<!--       <collision>
-        <origin xyz="0 0 ${0.008+0.095}" rpy="0 0 0"/>
-        <geometry>
-          <cylinder radius="0.006" length="0.016"/>
-        </geometry>
-        <material name="">
-          <color rgba="1 1 1 1"/>
-        </material>
-      </collision>  -->
     </link>
-    <joint name="$hand__end_effector_joint" type="fixed">
-      <parent link="ecpbi_base"/>
-      <child link="ecbpi_end_effector"/>
+    <joint name="${parent_link}_to_ecbpi_joint" type="fixed">
+      <parent link="${parent_link}"/>
+      <child link="ecbpi_base"/>
       <origin xyz="0 0 ${0.13}" rpy="0 0 0"/>
     </joint>
-    <link name="ecbpi_end_effector">
-      <gravity>0</gravity>
-      <visual>
-        <origin rpy="0 0 0.005" xyz="0 0 0"/>
-        <geometry>
-          <cylinder radius="0.0225" length="0.01"/>
-        </geometry>
-        <!-- <material name="transparent">
-          <color rgba="0 0 0 0"/>
-        </material> -->
-      </visual>
-      <inertial>
-        <origin rpy="0 0 0" xyz="0 0 0"/>
-        <mass value="0.0001"/>
-        <inertia ixx="1e-08" ixy="0" ixz="0" iyy="1e-08" iyz="0" izz="1e-08"/>
-      </inertial>
-    </link>
-    <xacro:epick_hand_gazebo robot_name="${robot_name}" />
+    <xacro:ecbpi_hand_gazebo robot_name="${robot_name}" />
   </xacro:macro>
 </robot>

File: tm_description/xacro/tm12_ecbpi.urdf (robot description, URDF)
Before this commit: robot tm12_ecpbi, 9 links, 8 joints
Links:
- added link ecbpi_base, mass 0.745; collision cylinder length=0.13 radius=0.044; visual cylinder length=0.03 radius=0.006
Joints:
- added joint flange_to_ecbpi_joint: type fixed, parent flange, child ecbpi_base, origin xyz=0 0 0.13 rpy=0 0 0

File: tm_description/xacro/tm12_ecbpi.urdf.xacro (robot description, xacro)
@@ -1,9 +1,8 @@
 <?xml version="1.0"?>
-<robot xmlns:xacro="http://www.ros.org/wiki/xacro" name="tm12_ecpbi">
+<robot xmlns:xacro="http://www.ros.org/wiki/xacro" name="tm12_ecbpi">
   <xacro:arg name="ns" default="" />
   <xacro:arg name="prefix" default="" />
   <xacro:arg name="color" default="none" />
   <xacro:arg name="trans_hw_iface" default="hardware_interface/PositionJointInterface" />
-  <xacro:arg name="hand_link_name" default="ecpbi_base" />
   <xacro:include filename="$(find tm_description)/xacro/macro.gazebo.xacro" />
   <xacro:include filename="$(find tm_description)/xacro/macro.transmission.xacro" />
@@ -13,5 +12,6 @@
   <!-- you must modify 'macro.tm12-nominal.urdf.xacro' to 'user_defined.urdf.xacro'  -->
   <xacro:include filename="$(find tm_description)/xacro/macro.tm12-nominal.urdf.xacro" />
-  <xacro:include filename="$(find tm_description)/xacro/schmalz_ecbpi_model_macro.xacro" />
+  <xacro:include filename="/home/tak-mahal/ws_moveit2/src/tmr_ros2/tm_description/xacro/schmalz_ecbpi_model_macro.xacro" />
+  <xacro:ecbpi_hand parent_link="flange" robot_name="tm12_ecbpi"/>
   <!--  -->
   <xacro:tmr_gazebo ns="$(arg ns)" prefix="$(arg prefix)" />
